Commit message: Add IMU sensor

File: quadrupedal_description/urdf/quadrupedal_robot.xacro (robot description, xacro)
@@ -77,4 +77,36 @@
 	<xacro:trans_macro name="upper_joint_trans4" joint_name="upper_joint4" act_name="upper_motor4"/>
 	<xacro:link_macro name="under_link4" ixx="0.000400596397" ixy="-0.000000183755" ixz="-0.000003142145" iyy="0.00040165997" iyz="-0.000020733392" izz="0.000006738557" mass="0.080527" filename="package://quadrupedal_description/meshes/stl/under_leg_left_ease_alt.stl" color="Blue"/>
+	<!--IMU-->
+	<joint name="imu_joint" type="fixed">
+		<parent link="body"/>
+		<child link="imu_link"/>
+		<origin xyz="0.15 0 0.6" rpy="0 0 0"/>
+	</joint>
+	<link name="imu_link"/>
+		<!--visual>
+			<geometry>
+				<box size="0.01 0.01 0.01"/>
+			</geometry>
+		</visual>
+	</link-->
+	<gazebo reference="imu_link">
+		<gravity>true</gravity>
+		<sensor name="imu_sensor" type="imu">
+			<always_on>true</always_on>
+			<update_rate>100</update_rate>
+			<visualize>true</visualize>
+			<topic>data</topic>
+			<plugin filename="libgazebo_ros_imu_sensor.so" name="imu_plugin">
+				<topicName>imu</topicName>
+				<bodyName>imu_link</bodyName>
+        <updateRateHZ>10.0</updateRateHZ>
+        <gaussianNoise>0.0</gaussianNoise>
+        <xyzOffset>0 0 0</xyzOffset>
+        <rpyOffset>0 0 0</rpyOffset>
+        <frameName>imu_link</frameName>
+			</plugin>
+			<pose>0 0 0 0 0 0</pose>
+		</sensor>
+	</gazebo>
 	<gazebo>
 		<plugin name="gazebo_ros_control" filename="libgazebo_ros_control.so">

Commit message: Add Depth Camera

File: quadrupedal_description/urdf/quadrupedal_robot.xacro (robot description, xacro)
@@ -81,13 +81,13 @@
 		<parent link="body"/>
 		<child link="imu_link"/>
-		<origin xyz="0.15 0 0.6" rpy="0 0 0"/>
+		<origin xyz="0.15 0 0.12" rpy="0 0 0"/>
 	</joint>
-	<link name="imu_link"/>
-		<!--visual>
+	<link name="imu_link">
+		<visual>
 			<geometry>
 				<box size="0.01 0.01 0.01"/>
 			</geometry>
 		</visual>
-	</link-->
+	</link>
 	<gazebo reference="imu_link">
 		<gravity>true</gravity>
@@ -109,4 +109,58 @@
 		</sensor>
 	</gazebo>
+	<!--Depth camera (unable)-->
+	<joint name="depth_camera_joint" type="fixed">
+		<parent link="body"/>
+		<child link="depth_link"/>
+		<origin xyz="0.21 0 0.06" rpy="0 0 0"/>
+	</joint>
+	<link name="depth_link">
+		<visual>
+			<geometry>
+				<box size="0.01 0.02 0.01"/>
+			</geometry>
+		</visual>
+	</link>
+	<gazebo reference="depth_link">
+  <sensor name="depth_camera" type="depth">
+    <update_rate>20</update_rate>
+    <camera>
+      <horizontal_fov>1.047198</horizontal_fov>
+      <image>
+        <width>640</width>
+        <height>480</height>
+        <format>R8G8B8</format>
+      </image>
+      <clip>
+        <near>0.05</near>
+        <far>3</far>
+      </clip>
+    </camera>
+    <plugin name="depth_camera_controller" filename="libgazebo_ros_openni_kinect.so">
+      <baseline>0.2</baseline>
+      <alwaysOn>true</alwaysOn>
+      <updateRate>1.0</updateRate>
+      <cameraName>depth_camera_ir</cameraName>
+      <imageTopicName>/depth_camera/depth/image_raw</imageTopicName>
+      <cameraInfoTopicName>/depth_camera/depth/camera_info</cameraInfoTopicName>
+      <depthImageTopicName>/depth_camera/depth/image_raw</depthImageTopicName>
+      <depthImageInfoTopicName>/depth_camera/depth/camera_info</depthImageInfoTopicName>
+      <pointCloudTopicName>/depth_camera/depth/points</pointCloudTopicName>
+      <frameName>depth_camera</frameName>
+      <pointCloudCutoff>0.5</pointCloudCutoff>
+      <pointCloudCutoffMax>3.0</pointCloudCutoffMax>
+      <distortionK1>0.00000001</distortionK1>
+      <distortionK2>0.00000001</distortionK2>
+      <distortionK3>0.00000001</distortionK3>
+      <distortionT1>0.00000001</distortionT1>
+      <distortionT2>0.00000001</distortionT2>
+      <CxPrime>0</CxPrime>
+      <Cx>0</Cx>
+      <Cy>0</Cy>
+      <focalLength>0</focalLength>
+      <hackBaseline>0</hackBaseline>
+    </plugin>
+  </sensor>
+</gazebo>
 	<gazebo>
 		<plugin name="gazebo_ros_control" filename="libgazebo_ros_control.so">

Commit message: Change the <mu>

File: quadrupedal_description/urdf/quadrupedal_robot.xacro (robot description, xacro)
@@ -19,6 +19,6 @@
 		</link>
 		<gazebo reference="${name}">
-			<mu1 value="0.5"/>
-			<mu2 value="0.4"/>
+			<mu1 value="0.8"/>
+			<mu2 value="0.8"/>
 			<material>Gazebo/${color}</material>
 		</gazebo>
@@ -30,6 +30,6 @@
 			<axis xyz="0 1 0"/>
 			<origin xyz="${x} ${y} ${z}" rpy="0 0 0"/>
-			<dynamics damping="0.05"/>
-			<limit lower="-1.57" upper="1.57" effort="6.0" velocity="6.0"/>
+			<dynamics damping="0.1"/>
+			<limit lower="-2.0" upper="2.0" effort="6.0" velocity="6.0"/>
 		</joint>
 	</xacro:macro>

Commit message: Add trj controller

File: quadrupedal_description/urdf/quadrupedal_robot.xacro (robot description, xacro)
@@ -19,6 +19,29 @@
 		</link>
 		<gazebo reference="${name}">
-			<mu1 value="0.8"/>
-			<mu2 value="0.8"/>
+			<mu1 value="100000.0"/>
+			<mu2 value="100000.0"/>
+			<material>Gazebo/${color}</material>
+		</gazebo>
+	</xacro:macro>
+	<xacro:macro name="tip_link_macro" params="name ixx ixy ixz iyy iyz izz mass filename color">
+		<link name="${name}">
+			<inertial>
+				<mass value="${mass}"/>
+				<inertia ixx="${ixx}" ixy="${ixy}"  ixz="${ixz}" iyy="${iyy}" iyz="${iyz}" izz="${izz}"/>
+			</inertial>
+			<visual>
+				<geometry>
+					<mesh filename="${filename}"/>
+				</geometry>
+			</visual>
+			<collision>
+				<geometry>
+					<mesh filename="${filename}"/>
+				</geometry>
+			</collision>
+		</link>
+		<gazebo reference="${name}">
+			<mu1 value="100000.0"/>
+			<mu2 value="100000.0"/>
 			<material>Gazebo/${color}</material>
 		</gazebo>
@@ -168,3 +191,11 @@
 		</plugin>
 	</gazebo>
+	<gazebo>
+		<plugin name="joint_state_publisher" filename="libgazebo_ros_joint_state_publisher.so">
+      <robotNamespace>/quadrupedal_robot</robotNamespace>
+      <jointName>body_joint1, body_joint2, body_joint3, body_joint4, upper_joint1, upper_joint2, upper_joint3, upper_joint4</jointName>
+      <updateRate>60.0</updateRate>
+      <alwaysOn>true</alwaysOn>
+    </plugin>
+  </gazebo>
 </robot>

Commit message: Update xacro

File: quadrupedal_description/urdf/quadrupedal_robot.xacro (robot description, xacro)
@@ -54,5 +54,5 @@
 			<origin xyz="${x} ${y} ${z}" rpy="0 0 0"/>
 			<dynamics damping="0.1"/>
-			<limit lower="-2.0" upper="2.0" effort="6.0" velocity="6.0"/>
+			<limit lower="-2.5" upper="2.5" effort="8.0" velocity="6.0"/>
 		</joint>
 	</xacro:macro>

Commit message: Change param

File: quadrupedal_description/urdf/quadrupedal_robot.xacro (robot description, xacro)
@@ -19,6 +19,6 @@
 		</link>
 		<gazebo reference="${name}">
-			<mu1 value="100000.0"/>
-			<mu2 value="100000.0"/>
+			<mu1 value="2000.0"/>
+			<mu2 value="1000.0"/>
 			<material>Gazebo/${color}</material>
 		</gazebo>
@@ -42,16 +42,18 @@
 		</link>
 		<gazebo reference="${name}">
-			<mu1 value="100000.0"/>
-			<mu2 value="100000.0"/>
+			<mu1 value="1000.0"/>
+			<mu2 value="2000.0"/>
+			<kp value="1000000"/>
+			<kd value="1.0"/>
 			<material>Gazebo/${color}</material>
 		</gazebo>
 	</xacro:macro>
-	<xacro:macro name="joint_macro" params="name x y z parent child">
-		<joint name="${name}" type="revolute">
+	<xacro:macro name="joint_macro" params="name x y z parent child type">
+		<joint name="${name}" type="${type}">
 			<parent link="${parent}"/>
 			<child link="${child}"/>
 			<axis xyz="0 1 0"/>
 			<origin xyz="${x} ${y} ${z}" rpy="0 0 0"/>
-			<dynamics damping="0.1"/>
+			<dynamics damping="0.05"/>
 			<limit lower="-2.5" upper="2.5" effort="8.0" velocity="6.0"/>
 		</joint>
@@ -76,26 +78,26 @@
 	</joint>
 	<xacro:link_macro name="body" ixx="0.013997409758" ixy="0.0"  ixz="0.0" iyy="0.032039793016" iyz="0.0" izz="0.029239204023" mass="1.43533" filename="package://quadrupedal_description/meshes/stl/body_assem_alt.stl" color="Blue"/>
-  <xacro:joint_macro name="body_joint1" x="0.15" y="-0.107" z="0.06" parent="body" child="upper_link1"/>
+  <xacro:joint_macro name="body_joint1" x="0.15" y="-0.107" z="0.06" parent="body" child="upper_link1" type="revolute"/>
 	<xacro:trans_macro name="body_joint_trans1" joint_name="body_joint1" act_name="body_motor1"/>
 	<xacro:link_macro name="upper_link1" ixx="0.0005696021" ixy="-0.000000000098" ixz="-0.000000000243" iyy="0.000513795097" iyz="0.000074601225" izz="0.000137674903" mass="0.307" filename="package://quadrupedal_description/meshes/stl/upper_leg_alt.stl" color="Red"/>
-	<xacro:joint_macro name="upper_joint1" x="0" y="0.00425" z="-0.130" parent="upper_link1" child="under_link1"/>
+	<xacro:joint_macro name="upper_joint1" x="0" y="0.00425" z="-0.130" parent="upper_link1" child="under_link1" type="revolute"/>
 	<xacro:trans_macro name="upper_joint_trans1" joint_name="upper_joint1" act_name="upper_motor1"/>
 	<xacro:link_macro name="under_link1" ixx="0.000400596397" ixy="0.000000183755" ixz="-0.000003142145" iyy="0.00040165997" iyz="0.000020733392" izz="0.000006738557" mass="0.080527" filename="package://quadrupedal_description/meshes/stl/under_leg_alt.stl" color="Blue"/>
-  <xacro:joint_macro name="body_joint2" x="-0.15" y="-0.107" z="0.06" parent="body" child="upper_link2"/>
+  <xacro:joint_macro name="body_joint2" x="-0.15" y="-0.107" z="0.06" parent="body" child="upper_link2" type="revolute"/>
 	<xacro:trans_macro name="body_joint_trans2" joint_name="body_joint2" act_name="body_motor2"/>
 	<xacro:link_macro name="upper_link2" ixx="0.0005696021" ixy="-0.000000000098" ixz="-0.000000000243" iyy="0.000513795097" iyz="0.000074601225" izz="0.000137674903" mass="0.307" filename="package://quadrupedal_description/meshes/stl/upper_leg_alt.stl" color="Red"/>
-	<xacro:joint_macro name="upper_joint2" x="0" y="0.00425" z="-0.130" parent="upper_link2" child="under_link2"/>
+	<xacro:joint_macro name="upper_joint2" x="0" y="0.00425" z="-0.130" parent="upper_link2" child="under_link2" type="revolute"/>
 	<xacro:trans_macro name="upper_joint_trans2" joint_name="upper_joint2" act_name="upper_motor2"/>
 	<xacro:link_macro name="under_link2" ixx="0.000400596397" ixy="0.000000183755" ixz="-0.000003142145" iyy="0.00040165997" iyz="0.000020733392" izz="0.000006738557" mass="0.080527" filename="package://quadrupedal_description/meshes/stl/under_leg_alt.stl" color="Blue"/>
-  <xacro:joint_macro name="body_joint3" x="-0.15" y="0.107" z="0.06" parent="body" child="upper_link3"/>
+  <xacro:joint_macro name="body_joint3" x="-0.15" y="0.107" z="0.06" parent="body" child="upper_link3" type="revolute"/>
 	<xacro:trans_macro name="body_joint_trans3" joint_name="body_joint3" act_name="body_motor3"/>
 	<xacro:link_macro name="upper_link3" ixx="0.000569601994" ixy="0.0000000001" ixz="-0.000000000243" iyy="0.000513795026" iyz="-0.000074601184" izz="0.000137674854" mass="0.307" filename="package://quadrupedal_description/meshes/stl/upper_leg_left_ease_alt.stl" color="Red"/>
-	<xacro:joint_macro name="upper_joint3" x="0" y="-0.00425" z="-0.130" parent="upper_link3" child="under_link3"/>
+	<xacro:joint_macro name="upper_joint3" x="0" y="-0.00425" z="-0.130" parent="upper_link3" child="under_link3" type="revolute"/>
 	<xacro:trans_macro name="upper_joint_trans3" joint_name="upper_joint3" act_name="upper_motor3"/>
 	<xacro:link_macro name="under_link3" ixx="0.000400596397" ixy="-0.000000183755" ixz="-0.000003142145" iyy="0.00040165997" iyz="-0.000020733392" izz="0.000006738557" mass="0.080527" filename="package://quadrupedal_description/meshes/stl/under_leg_left_ease_alt.stl" color="Blue"/>
-  <xacro:joint_macro name="body_joint4" x="0.15" y="0.107" z="0.06" parent="body" child="upper_link4"/>
+  <xacro:joint_macro name="body_joint4" x="0.15" y="0.107" z="0.06" parent="body" child="upper_link4" type="revolute"/>
 	<xacro:trans_macro name="body_joint_trans4" joint_name="body_joint4" act_name="body_motor4"/>
 	<xacro:link_macro name="upper_link4" ixx="0.000569601994" ixy="0.0000000001" ixz="-0.000000000243" iyy="0.000513795026" iyz="-0.000074601184" izz="0.000137674854" mass="0.307" filename="package://quadrupedal_description/meshes/stl/upper_leg_left_ease_alt.stl" color="Red"/>
-	<xacro:joint_macro name="upper_joint4" x="0" y="-0.00425" z="-0.130" parent="upper_link4" child="under_link4"/>
+	<xacro:joint_macro name="upper_joint4" x="0" y="-0.00425" z="-0.130" parent="upper_link4" child="under_link4" type="revolute"/>
 	<xacro:trans_macro name="upper_joint_trans4" joint_name="upper_joint4" act_name="upper_motor4"/>
 	<xacro:link_macro name="under_link4" ixx="0.000400596397" ixy="-0.000000183755" ixz="-0.000003142145" iyy="0.00040165997" iyz="-0.000020733392" izz="0.000006738557" mass="0.080527" filename="package://quadrupedal_description/meshes/stl/under_leg_left_ease_alt.stl" color="Blue"/>
